File: cycfi-nu-hub/cycfi-nu-hub.kicad_pcb (KiCad board)
At the start: 2 copper layers, 61 x 24 mm, 18 parts, among them J1 TO BREAKOUT J3, P1 CH1 PWR, P2 CH2 PWR, P3 CH3 PWR, P4 CH4 PWR, P5 CH5 PWR, P6 CH6 PWR

Commit message: Clarified E1 shield
Parts:
- E1: value BRIDGE/SHIELD -> SHIELD/GND
Other:
- board text added: "GND"
- board text removed: "BRIDGE"
