File: cycfi-nu-hub/cycfi-nu-hub.kicad_sch (KiCad schematic)
At the start: 18 parts, among them J1 TO BREAKOUT J3, P1 CH1 PWR, P2 CH2 PWR, P3 CH3 PWR, P4 CH4 PWR, P5 CH5 PWR, P6 CH6 PWR

Commit message: Added instructions on how to make the cables
Other:
- note added: "Bridge earth or cavity foil. Optional -- see docs/DESIGN.md."
- note removed: "Bridge earth or cavity foil. Optional -- see DESIGN.md."
Changed lines of the file:
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@@
 		)
 	)
-	(text "Bridge earth or cavity foil. Optional -- see DESIGN.md."
+	(text "Bridge earth or cavity foil. Optional -- see docs/DESIGN.md."
 		(at 53.34 215.9 0)
 		(effects

Commit message: Clarified E1 shield
Parts:
- E1: value BRIDGE/SHIELD -> SHIELD/GND
Other:
- note added: "Trunk cable screen; cavity foil. See docs/DESIGN.md."
- note removed: "Bridge earth or cavity foil. Optional -- see docs/DESIGN.md."
Changed lines of the file:
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@@
 		)
 	)
-	(text "Bridge earth or cavity foil. Optional -- see docs/DESIGN.md."
+	(text "Trunk cable screen; cavity foil. See docs/DESIGN.md."
 		(at 53.34 215.9 0)
 		(effects
@@
 			)
 		)
-		(property "Value" "BRIDGE/SHIELD"
+		(property "Value" "SHIELD/GND"
 			(at 45.72 222.25 0)
 			(effects
@@
 			)
 		)
-		(property "Description" "Solder pad to GND for bridge earth or cavity shielding, 1.0mm hole"
+		(property "Description" "Solder pad to GND: trunk cable screen, cavity foil, optionally bridge earth"
 			(at 45.72 215.9 0)
 			(effects
