File: cycfi-nu-hub/cycfi-nu-hub.kicad_sch (KiCad schematic)
At the start: 18 parts, among them J1 TO BREAKOUT J3, P1 CH1 PWR, P2 CH2 PWR, P3 CH3 PWR, P4 CH4 PWR, P5 CH5 PWR, P6 CH6 PWR

Commit message: Match the Internal Breakout's outline and hole pattern
The hub was a 61 x 24 mm strip of its own choosing. It is now 50 x 35 mm with
1.75 mm corners and four M2 holes on 45 x 30 mm centres -- the breakout's own
geometry -- so one mount, one cavity cut-out or one enclosure pocket takes
either board.

Every number is measured off Cycfi's internal_breakout.brd (Eagle layer 20)
and lives in design.MOUNTING_PATTERN; gen_pcb.py derives its dimensions from
there and asserts the hole centres against it. Two figures are deliberately
regularised rather than transcribed, and both are recorded: Cycfi's four hole
centres are not quite a rectangle (29.9 vs 30.0 mm, insets 2.52 to 2.55), and
their four corner arcs do not share a radius (three at ~1.77, one at 1.63).

Also corrects a misattribution in the docs. They stated Cycfi list breakout
v2.6 as 27 x 38 mm; that figure is prose from the Nu Series *v1* page and
names no version. The v2.6.1 datasheet carries no dimensions at all and
neither does the 2023 redesign announcement, so 50 x 35 is the only measured
breakout outline in existence -- and it is v2.5's. That assumption now travels
with the geometry in fab/*-mechanical.json rather than living only in prose.

Three things fell out of the smaller outline:

- The fan-in had to be re-derived. The lanes stay north of the signal row, and
  check_placement() now asserts the lane order and descent order are reverses
  of each other -- the property that was violated when the middle band looked
  like the obvious home for them.
- check_holes_clear() is new. At 2.5 mm in from all four edges the holes now
  sit in the margin the descents run down, and an unplated hole has no pad, no
  net and no courtyard, so nothing else here would notice a track across one.
- check_fits() tests courtyard polygons against the rounded outline. Bounding
  boxes falsely reported all four holes as overhanging a board they fit.

ERC 0, DRC 0 (warnings included), netlist matches design.py.

Co-Authored-By: C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
Parts:
- H1, H2, H3, H4: value M2.5 -> M2; footprint MountingHole:MountingHole_2.7mm_M2.5 -> MountingHole:MountingHole_2.2mm_M2
Changed lines of the file:
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@@
 			)
 		)
-		(property "Value" "M2.5"
+		(property "Value" "M2"
 			(at 152.4 247.65 0)
 			(effects
@@
 			)
 		)
-		(property "Footprint" "MountingHole:MountingHole_2.7mm_M2.5"
+		(property "Footprint" "MountingHole:MountingHole_2.2mm_M2"
 			(at 152.4 241.3 0)
 			(effects
@@
 			)
 		)
-		(property "Description" "M2.5 clearance hole, unplated"
+		(property "Description" "M2 clearance hole, unplated"
 			(at 152.4 241.3 0)
 			(effects
@@
 			)
 		)
-		(property "Value" "M2.5"
+		(property "Value" "M2"
 			(at 165.1 247.65 0)
 			(effects
@@
 			)
 		)
-		(property "Footprint" "MountingHole:MountingHole_2.7mm_M2.5"
+		(property "Footprint" "MountingHole:MountingHole_2.2mm_M2"
 			(at 165.1 241.3 0)
 			(effects
@@
 			)
 		)
-		(property "Description" "M2.5 clearance hole, unplated"
+		(property "Description" "M2 clearance hole, unplated"
 			(at 165.1 241.3 0)
 			(effects
@@
 			)
 		)
-		(property "Value" "M2.5"
+		(property "Value" "M2"
 			(at 177.8 247.65 0)
 			(effects
@@
 			)
 		)
-		(property "Footprint" "MountingHole:MountingHole_2.7mm_M2.5"
+		(property "Footprint" "MountingHole:MountingHole_2.2mm_M2"
 			(at 177.8 241.3 0)
 			(effects
@@
 			)
 		)
-		(property "Description" "M2.5 clearance hole, unplated"
+		(property "Description" "M2 clearance hole, unplated"
 			(at 177.8 241.3 0)
 			(effects
@@
 			)
 		)
-		(property "Value" "M2.5"
+		(property "Value" "M2"
 			(at 190.5 247.65 0)
 			(effects
@@
 			)
 		)
-		(property "Footprint" "MountingHole:MountingHole_2.7mm_M2.5"
+		(property "Footprint" "MountingHole:MountingHole_2.2mm_M2"
 			(at 190.5 241.3 0)
 			(effects
@@
 			)
 		)
-		(property "Description" "M2.5 clearance hole, unplated"
+		(property "Description" "M2 clearance hole, unplated"
 			(at 190.5 241.3 0)
 			(effects

Commit message: Add a direct variant that replaces the Internal Breakout
For an installation that uses none of the breakout's aux, CV, GK or
power-select features, the breakout is a wire and a fuse. Every channel net in
Cycfi's internal_breakout.sch has exactly two pins on it -- the Nu Multi input
and the 19-pin jack -- with no buffer, filter or protection between them. So
the hub can drive the jack itself and take a board out of the chain.

    ./build.sh          the breakout-facing board, unchanged
    ./build.sh direct   35 x 24.5 mm, straight to the 19-pin jack

The capsule end of both is identical. design.VARIANT picks between them and
everything downstream follows: project name, fab filenames, which ORDER.md
verify.py asserts against.

Three findings make it tractable, all recorded in docs/cycfi-sources.md:

- The jack is two 2x5 headers, J10 and J11, so the hub presents the same pair
  the breakout does and the instrument's existing loom plugs in unmodified.
- There is no regulator to reproduce. Cycfi deleted theirs in v2.6 because the
  capsules run from 5 V to 18 V, which also settles the old open question
  about what voltage six of them would see.
- Reverse protection is already at every load; each capsule has its own
  Schottky. The breakout's P-FET protected the breakout's own regulator.

Two components, and NO_COMPONENTS is reopened rather than deleted. Its
argument rejects shunt parts a cable's length from their load, and neither of
these is that: F1 is in series, so what it protects is the run it is in, and
C1 is bulk where power enters the board. check_no_components() now enforces
exactly ['C1', 'F1'] on this variant -- a third part means the argument was
stretched rather than met. F1's 50 mA hold is a decision, not a transcription:
Cycfi's 500 mA has to pass aux loads and fifteen channels, and six capsules
draw about 1 mA each.

One safety property regresses and is documented rather than designed away. On
the breakout board a reversed 2x5 is harmless by construct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
Other:
- note added: "M2 clearance, unplated -- not on GND"
- note added: "No supply on this board: every rail arrives on J1."
- note removed: "M2.5 clearance, unplated -- not on GND"
- note removed: "No supply on this board: both rails arrive on J1."
Changed lines of the file:
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@@
 		)
 	)
-	(text "M2.5 clearance, unplated -- not on GND"
+	(text "M2 clearance, unplated -- not on GND"
 		(at 151.13 250.19 0)
 		(effects
@@
 		)
 	)
-	(text "No supply on this board: both rails arrive on J1."
+	(text "No supply on this board: every rail arrives on J1."
 		(at 40.64 234.95 0)
 		(effects
